File: pcb/esp32.kicad_pcb (KiCad board)
At the start: 2 copper layers, 13 parts, among them Q1 BC817, U1 ESP32-WROOM-32

Commit message: added some componentes to schematics and pcb
Parts:
- removed C2: 10u, Capacitor_SMD:CP_Elec_5x3
- removed C3: 50n, Capacitor_SMD:C_0805_2012Metric_Pad1.18x1.45mm_HandSolder
- removed RV5: 10K, Potentiometer_SMD:Potentiometer_Bourns_3314G_Vertical
- added J1: Conn_01x04, Connector_PinHeader_2.54mm:PinHeader_1x04_P2.54mm_Horizontal, F.Cu at (256.5, 123.2)
- added J10: Conn_01x02, Connector_PinHeader_2.54mm:PinHeader_1x02_P2.54mm_Vertical, F.Cu at (38.1, 137.2)
- added J11: Conn_01x02, Connector_PinHeader_2.54mm:PinHeader_1x02_P2.54mm_Vertical, F.Cu at (38.1, 116.8)
- added J12: Conn_01x05, Connector_PinHeader_2.54mm:PinHeader_1x05_P2.54mm_Vertical, F.Cu at (18.8, 121.9)
- added J13: Conn_01x02, Connector_PinHeader_2.54mm:PinHeader_1x02_P2.54mm_Vertical, F.Cu at (25.4, 121.9)
- added J14: Conn_01x02, Connector_PinHeader_2.54mm:PinHeader_1x02_P2.54mm_Vertical, F.Cu at (25.4, 129.5)
- added J2: Conn_01x01, Connector_PinHeader_2.54mm:PinHeader_1x01_P2.54mm_Vertical, F.Cu at (248.9, 116.8)
- added J3: Conn_01x01, Connector_PinHeader_2.54mm:PinHeader_1x01_P2.54mm_Vertical, F.Cu at (48.3, 116.8)
- added J4: Conn_01x01, Connector_PinHeader_2.54mm:PinHeader_1x01_P2.54mm_Vertical, F.Cu at (48.3, 123.2)
- added J5: Conn_01x01, Connector_PinHeader_2.54mm:PinHeader_1x01_P2.54mm_Vertical, F.Cu at (248.9, 123.2)
- added J6: Conn_01x01, Connector_PinHeader_2.54mm:PinHeader_1x01_P2.54mm_Vertical, F.Cu at (48.3, 130.8)
- added J7: Conn_01x01, Connector_PinHeader_2.54mm:PinHeader_1x01_P2.54mm_Vertical, F.Cu at (248.9, 130.8)
- added J8: Conn_01x01, Connector_PinHeader_2.54mm:PinHeader_1x01_P2.54mm_Vertical, F.Cu at (48.3, 137.2)
- added J9: Conn_01x01, Connector_PinHeader_2.54mm:PinHeader_1x01_P2.54mm_Vertical, F.Cu at (248.9, 137.2)
- added Q2: BC817, Package_TO_SOT_SMD:SOT-23_Handsoldering, B.Cu at (238.8, 123.2)
- added Q3: BC817, Package_TO_SOT_SMD:SOT-23_Handsoldering, B.Cu at (238.8, 130.8)
- added Q4: BC817, Package_TO_SOT_SMD:SOT-23_Handsoldering, B.Cu at (238.8, 137.2)
- added R3: 1K, Resistor_SMD:R_0805_2012Metric_Pad1.20x1.40mm_HandSolder, B.Cu at (245.1, 116.8)
- added R4: 1K, Resistor_SMD:R_0805_2012Metric_Pad1.20x1.40mm_HandSolder, B.Cu at (245.1, 123.2)
- added R5: 1K, Resistor_SMD:R_0805_2012Metric_Pad1.20x1.40mm_HandSolder, B.Cu at (245.1, 130.8)
- added R6: 1K, Resistor_SMD:R_0805_2012Metric_Pad1.20x1.40mm_HandSolder, B.Cu at (245.1, 137.2)
- added R7: 1K, Resistor_SMD:R_0805_2012Metric_Pad1.20x1.40mm_HandSolder, B.Cu at (30.5, 132.1)
- C1, C4, Q1, R1, R2, U1: moved to B.Cu
- moved RV1 212.7 mm to (274.6, 133.4), turned to 103 degrees
- moved RV2 207.9 mm to (279.4, 121.3), turned to -103 degrees
- moved RV3 184.3 mm to (262.0, 116.8), turned to -103 degrees
- moved RV4 181.5 mm to (257.2, 137.6), turned to 103 degrees
- moved Q1 169.5 mm to (238.8, 116.8), turned to 180 degrees
- moved U1 92.2 mm to (213.4, 124.5)
- moved R1 82.3 mm to (190.5, 130.8), turned to 90 degrees
- moved C1 81.6 mm to (190.5, 126.0), turned to 90 degrees
- moved R2 56.2 mm to (30.5, 129.5), turned to 180 degrees
- moved C4 45.7 mm to (36.8, 127.0), turned to -90 degrees
Connections:
- net /ADC1_CH6 renamed /Potis/ADC1_CH6
- net /ADC1_CH7 renamed /Potis/ADC1_CH7
- C4 pad 2: SPEAKER -> Net-(C4-Pad2)
- Q1 pad 1: SAITE_1 -> Net-(Q1-B)
- R2 pad 1: Net-(C3-Pad2) -> Net-(C4-Pad2)
- RV1 pad 2: /ADC1_CH0 -> /Potis/ADC1_CH0
- RV2 pad 2: /ADC1_CH3 -> /Potis/ADC1_CH3
Routing:
- net GND: track 0.00 -> 425.7 mm, vias 0 -> 4
- net DAC1: track 0.00 -> 180.0 mm
- net +3.3V: track 0.00 -> 73.3 mm
- net DIN4: track 0.00 -> 21.5 mm
- net DIN3: track 0.00 -> 18.6 mm
- net Net-(U1-EN): track 0.00 -> 17.1 mm
- net DIN2: track 0.00 -> 16.4 mm
- net DIN1: track 0.00 -> 16.0 mm
- net Net-(J10-Pin_1): track 0.00 -> 13.8 mm
- net Net-(J13-Pin_2): track 0.00 -> 11.6 mm
- net Net-(C4-Pad2): track 0.00 -> 5.81 mm
- net Net-(Q2-B): track 0.00 -> 4.24 mm
- net Net-(Q1-B): track 0.00 -> 4.24 mm
- net Net-(Q4-B): track 0.00 -> 4.24 mm
- net Net-(Q3-B): track 0.00 -> 4.24 mm
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Other:
- board outline added: 271.8 x 30.5 mm
